File: Hardware/Waveform_generator_faceplates/Waveform_generator_faceplates.kicad_sch (KiCad schematic)
At the start: 8 parts

Commit message: Revisión 1 del hardware. Reorganizaco un poco el layout y añadidos shottky de protección, puente para desconectar el buck, conectores de pogo para conectar a masa la carcasa de aluminio, agrandado el espacio del powerOpAmp para un mayor disipador...
Actualizado el controlador para que por USB no printee la batería todo el rato.

Añadida opción de reseteo del AD9837 en cada comando para probar si se soluciona el problema  (no genera nada a la salida)
Parts:
- added TP1: TP, TestPoint:TestPoint_THTPad_D2.0mm_Drill1.0mm, symbol Connector:TestPoint
- H1, H2, H3, H4, H5, H6, H7, H8: footprint MountingHole:MountingHole_2.2mm_M2_Pad_TopBottom -> CUSTOM:M3 hole (3.2mm hole Pad 5mm)
Connections:
- net GND: now also TP1.1; no longer H5.1, H6.1, H7.1, H8.1
- new net GND1: H5.1, H6.1, H7.1, H8.1
