File: Hardware/Waveform_generator/Waveform_generator.kicad_sch (KiCad schematic)
At the start: 106 parts, among them J1 Conn_01x02, J2 Conn_01x02, J3 Conn_01x02, J4 Conn_01x02, J5 PogoPin, J6 PogoPin, J7 GND_CHASIS, J8 GND_CHASIS, Q1 WSD4070DN33, Q2 WSD4070DN33, Q3 TLP3906TPL_E, Q4 MMBT3904, SW1 SW_DPDT_x2, U1 TPS54202DDC, U10 MCP4822, U11 LM1875, U2 TL072, U3 ESP32-DEVKITC-32U, U5 XC6206PxxxMR, U6 AD9837BCPZ-RL7, U7 TL072, U8 AD5160, U9 TL072, Y1 X1G0041710027

Commit message: pequeños cambios
Connections:
- net at Q1.5 (D), U11.4: no longer R24.2, R25.2
- new net: R24.2, R25.2
Other:
- moved on the sheet: C1, C11, C12, C17, C18, C19, C2, C20, C3, C4, C5, C6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
